Commit message: fixed sim toppling

File: calypso-simulator/calypso_sim/model/auv.urdf.xacro (robot description, xacro)
@@ -49,5 +49,5 @@
       <inertial>
         <mass value="160"/>
-        <inertia ixx="466338.03533197" ixy="0.00022747" ixz="-0.00184206" iyy="846140.53520644" iyz="-13851.49143136" izz="547835.76597596"/>
+        <inertia ixx="0" ixy="0" ixz="0" iyy="0" iyz="0" izz="0"/>
       </inertial>
     </link>

Commit message: kinda fixed simulator

File: calypso-simulator/calypso_sim/model/auv.urdf.xacro (robot description, xacro)
@@ -21,6 +21,6 @@
     <!-- <xacro:property name="x" default="0"/>
     <xacro:property name="y" default="0"/> -->
-    <xacro:property name="x" default="-0.35"/>
-    <xacro:property name="y" default="0.35"/>
+    <xacro:property name="x" default="-0.26"/>
+    <xacro:property name="y" default="0.43"/>
     <xacro:property name="z" default="0"/>
     <xacro:property name="r" default="1.57"/>
@@ -32,23 +32,25 @@
         <parent link="dummy"/>
         <child link="base_link"/>
-        <origin xyz="${x} ${y} ${z}" rpy="${r} ${p} ${Y}"/>
+        <origin xyz="0 0 0" rpy="${r} ${p} ${Y}"/>
     </joint> -->
     <link name="base_link">
         <visual>
           <geometry>
-              <mesh filename="package://calypso_sim/meshes/auv-body/auv.STL" scale="0.001 0.001 0.001"/>
+              <mesh filename="package://calypso_sim/meshes/auv-body/AUV.STL" scale="0.001 0.001 0.001"/>
           </geometry>
-          <origin xyz="${x} ${y} ${z}" rpy="${r} ${p} ${Y}" />
+          <origin xyz="0 0 0" rpy="${r} ${p} ${Y}" />
           <material name="yellow"/>
       </visual>
       <collision>
         <geometry>
-          <mesh filename="package://calypso_sim/meshes/auv-body/auv.STL" scale="0.001 0.001 0.001"/>
+          <origin xyz="0 0 0" rpy="${r} ${p} ${Y}" />
+          <mesh filename="package://calypso_sim/meshes/auv-body/AUV.STL" scale="0.001 0.001 0.001"/>
         </geometry>
       </collision>
-      <inertial>
-        <mass value="160"/>
-        <inertia ixx="0" ixy="0" ixz="0" iyy="0" iyz="0" izz="0"/>
-      </inertial>
+    <inertial>
+      <mass value="37.00000000"/>
+      <inertia ixx="1002084.26190628" ixy="-0.00000934" ixz="-0.00004849" iyy="1472890.49211890" iyz="1402.25179064" izz="689649.10160904"/>
+      <!-- <inertia ixx="0" ixy="0" ixz="0" iyy="0" iyz="0" izz="0"/> -->
+    </inertial>
     </link>
     <gazebo reference="base_link">
@@ -65,23 +67,25 @@
 -->
     <!-- ${x}-0.32 ${y}-0.06 ${z}+0.1 -->
-    <xacro:thruster_CCW id="1" parent="base_link" xyz="0.26 -0.062 0.1" rpy="0 0 0" axis="0 0 -1">
+    <xacro:thruster_CCW id="1" parent="base_link" xyz="0.445 -0.54 0.25" rpy="0 0 0" axis="0 0 -1">
     </xacro:thruster_CCW>
-    <xacro:thruster_CW id="2" parent="base_link" xyz="${x-x-0.32} ${y-y-0.06} ${z+0.1}" rpy="0 0 0" axis="0 0 1">
+    <xacro:thruster_CW id="2" parent="base_link" xyz="0.06 -0.54 0.25" rpy="0 0 0" axis="0 0 1">
     </xacro:thruster_CW>
-    <xacro:thruster_CW id="4" parent="base_link" xyz="0.26 0.12 0.1" rpy="0 0 0" axis="0 0 1">
+    <xacro:thruster_CW id="4" parent="base_link" xyz="0.445 -0.32 0.25" rpy="0 0 0" axis="0 0 1">
     </xacro:thruster_CW>
-    <xacro:thruster_CCW id="3" parent="base_link" xyz="-0.32 0.12 0.1" rpy="0 0 0" axis="0 0 -1" >
+    <xacro:thruster_CCW id="3" parent="base_link" xyz="0.06 -0.32 0.25" rpy="0 0 0" axis="0 0 -1" >
     </xacro:thruster_CCW>
-    <xacro:thruster_CCW id="5" parent="base_link" xyz="0.22 -0.22 0.06" rpy="0 1.57 0.785" axis="0 0 -1">
+    <xacro:property name="x" default="-0.26"/>
+    <xacro:property name="y" default="0.43"/>
+    <xacro:thruster_CCW id="5" parent="base_link" xyz="0.41 -0.68 0.17" rpy="0 1.57 0.785398" axis="0 0 -1">
     </xacro:thruster_CCW>
-    <xacro:thruster_CW id="6" parent="base_link" xyz="-0.23 -0.23 0.06" rpy="0 1.57 2.182" axis="0 0 1">
+    <xacro:thruster_CW id="6" parent="base_link" xyz="0.11 -0.68 0.17" rpy="0 1.57 2.35619" axis="0 0 1">
     </xacro:thruster_CW>
-    <xacro:thruster_CCW id="7" parent="base_link" xyz="-0.26 0.28 0.06" rpy="0 1.57 3.92" axis="0 0 -1">
+    <xacro:thruster_CCW id="7" parent="base_link" xyz="0.11 -0.18 0.17" rpy="0 1.57 3.92" axis="0 0 -1">
     </xacro:thruster_CCW>
-    <xacro:thruster_CW id="8" parent="base_link" xyz="0.22 0.28 0.06" rpy="0 1.57 -0.785" axis="0 0 1">
+    <xacro:thruster_CW id="8" parent="base_link" xyz="0.41 -0.18 0.17" rpy="0 1.57 -0.785398" axis="0 0 1">
     </xacro:thruster_CW>
-    <xacro:camera id="1" parent="base_link" xyz="-0.02 -0.2 0.19" rpy="0 0 -1.57">
+    <xacro:camera id="1" parent="base_link" xyz="0.255 -0.68 0.25" rpy="0 0 -1.57">
     </xacro:camera>
-    <xacro:imu id="1" parent="base_link" xyz="-0.02 0.1 0.06" rpy="0 0 -1.57">
+    <xacro:imu id="1" parent="base_link" xyz="0.24 -0.4 0.25" rpy="0 0 -1.57">
     </xacro:imu>
     <gazebo>
@@ -91,11 +95,26 @@
       </plugin>
     </gazebo>
-    <gazebo>
-      <plugin name="BuoyancyPlugin" filename="libBuoyancyPlugin.so">
-        <fluid_density>1000</fluid_density>
-        <link name="base_link">
-          <volume>0.00964522875</volume>
-        </link>
-      </plugin>
-    </gazebo>
+  <!-- <gazebo>
+    <plugin name="freebuoyancy_gazebo" filename="libfreebuoyancy_gazebo.so">
+      <descriptionParam>robot_description</descriptionParam>
+      <alwaysOn>true</alwaysOn>
+      <surface>0 0 0</surface>
+      <updateRate>.001</updateRate>
+      <link name='base_link'>
+        <buoyancy>
+          <compensation>0</compensation>
+          <origin xyz="0 0 0"/>
+        </buoyancy>
+      </link>
+    </plugin>
+  </gazebo> -->
+  <gazebo>
+     <plugin name="BuoyancyPlugin" filename="libBuoyancyPlugin.so">
+      <fluid_density>1000</fluid_density>
+      <link name="base_link">
+        <volume>0.03</volume>
+        <center_of_volume>0 0 0</center_of_volume>
+      </link>
+    </plugin>
+  </gazebo>
 </robot>

File: calypso-simulator/calypso_sim/model/thrusters.urdf.xacro (robot description, xacro)
@@ -8,5 +8,5 @@
         <material name="red"/>
         <geometry>
-           <mesh filename="${thrusterCCW_path}T200_Thruster.dae" scale="1.5 1.5 1.5"/>
+           <mesh filename="${thrusterCCW_path}T200_Thruster.dae" scale="1 1 1"/>
            <!--<box size="0.1 0.1 0.1"/>-->
         </geometry>
@@ -14,5 +14,5 @@
       <collision>
         <geometry>
-          <mesh filename="${thrusterCCW_path}T200_Thruster.dae" scale="1.5 1.5 1.5"/>
+          <mesh filename="${thrusterCCW_path}T200_Thruster.dae" scale="1 1 1"/>
         </geometry>
       </collision>
@@ -34,10 +34,10 @@
       <visual>
         <geometry>
-          <mesh filename="${thrusterCCW_path}T200_Prop_CCW.dae" scale="1.5 1.5 1.5"/>
-        </geometry>
-      </visual>
-      <collision>
-        <geometry>
-          <mesh filename="${thrusterCCW_path}T200_Prop_CCW.dae" scale="1.5 1.5 1.5"/>
+          <mesh filename="${thrusterCCW_path}T200_Prop_CCW.dae" scale="1 1 1"/>
+        </geometry>
+      </visual>
+      <collision>
+        <geometry>
+          <mesh filename="${thrusterCCW_path}T200_Prop_CCW.dae" scale="1 1 1"/>
         </geometry>
       </collision>
@@ -96,4 +96,15 @@
       <allow_auto_disable>0</allow_auto_disable>
     </gazebo>
+    <!-- <gazebo>
+      <plugin name="freefloating_gazebo_control" filename="libfreefloating_gazebo_control.so">
+        <switchService>switch</switchService>
+        <updateRate>100</updateRate>
+        <link>base_link</link>
+        <thruster>
+            <map>${xyz} ${rpy}</map>
+            <effort>30</effort>
+        </thruster>
+      </plugin>
+    </gazebo> -->
      <gazebo reference="prop_${id}">
         <material>Gazebo/Red</material>
@@ -104,5 +115,5 @@
        <visual>
         <geometry>
-           <mesh filename="${thrusterCW_path}T200_Thruster.dae" scale="1.5 1.5 1.5"/>
+           <mesh filename="${thrusterCW_path}T200_Thruster.dae" scale="1 1 1"/>
            <!--<box size="0.1 0.1 0.1"/>-->
         </geometry>
@@ -111,5 +122,5 @@
       <collision>
         <geometry>
-          <mesh filename="${thrusterCW_path}T200_Thruster.dae" scale="1.5 1.5 1.5"/>
+          <mesh filename="${thrusterCW_path}T200_Thruster.dae" scale="1 1 1"/>
         </geometry>
       </collision>
@@ -131,5 +142,5 @@
       <visual>
         <geometry>
-          <mesh filename="${thrusterCW_path}T200_Prop_CW.dae" scale="1.5 1.5 1.5"/>
+          <mesh filename="${thrusterCW_path}T200_Prop_CW.dae" scale="1 1 1"/>
         </geometry>
         <material name="green"/>
@@ -137,5 +148,5 @@
       <collision>
         <geometry>
-          <mesh filename="${thrusterCW_path}T200_Prop_CW.dae" scale="1.5 1.5 1.5"/>
+          <mesh filename="${thrusterCW_path}T200_Prop_CW.dae" scale="1 1 1"/>
         </geometry>
       </collision>
@@ -194,6 +205,17 @@
       <allow_auto_disable>0</allow_auto_disable>
     </gazebo>
-     <gazebo reference="prop_${id}">
-        <material>Gazebo/Green</material>
+  <!-- <gazebo>
+      <plugin name="freefloating_gazebo_control" filename="libfreefloating_gazebo_control.so">
+        <switchService>switch</switchService>
+        <updateRate>100</updateRate>
+        <link>base_link</link>
+        <thruster>
+            <map>-1 0 0 0 0 ${-body_width/2}</map>
+            <effort>30</effort>
+        </thruster>
+      </plugin>
+  </gazebo> -->
+    <gazebo reference="prop_${id}">
+      <material>Gazebo/Green</material>
     </gazebo>
   </xacro:macro>

Commit message: cleaned up

File: calypso-simulator/calypso_sim/model/auv.urdf.xacro (robot description, xacro)
@@ -109,12 +109,3 @@
     </plugin>
   </gazebo>
-  <gazebo>
-     <!-- <plugin name="BuoyancyPlugin" filename="libBuoyancyPlugin.so">
-      <fluid_density>1000</fluid_density>
-      <link name="base_link">
-        <volume>0.03</volume>
-        <center_of_volume>0 0 0</center_of_volume>
-      </link>
-    </plugin>
-  </gazebo> -->
 </robot>

Commit message: simulator reverted to old version

File: calypso-simulator/calypso_sim/model/auv.urdf.xacro (robot description, xacro)
@@ -4,4 +4,5 @@
     <xacro:include filename="$(find calypso_sim)/model/imu.urdf.xacro"/>
     <xacro:include filename="$(find calypso_sim)/model/thrusters.urdf.xacro"/>
+    <xacro:include filename="$(find calypso_sim)/model/chasis.urdf.xacro"/>
     <material name="red">
         <color rgba="1 0 0 1"/>
@@ -27,34 +28,5 @@
     <xacro:property name="p" default="0"/>
     <xacro:property name="Y" default="0"/>
-    <!-- <link name="dummy">
-    </link>
-    <joint name="base_link_to_dummy" type="fixed">
-        <parent link="dummy"/>
-        <child link="base_link"/>
-        <origin xyz="0 0 0" rpy="${r} ${p} ${Y}"/>
-    </joint> -->
-    <link name="base_link">
-        <visual>
-          <geometry>
-              <mesh filename="package://calypso_sim/meshes/auv-body/AUV.STL" scale="0.001 0.001 0.001"/>
-          </geometry>
-          <origin xyz="0 0 0" rpy="${r} ${p} ${Y}" />
-          <material name="yellow"/>
-      </visual>
-      <collision>
-        <geometry>
-          <origin xyz="0 0 0" rpy="${r} ${p} ${Y}" />
-          <mesh filename="package://calypso_sim/meshes/auv-body/AUV.STL" scale="0.001 0.001 0.001"/>
-        </geometry>
-      </collision>
-    <inertial>
-      <mass value="37.00000000"/>
-      <inertia ixx="1002084.26190628" ixy="-0.00000934" ixz="-0.00004849" iyy="1472890.49211890" iyz="1402.25179064" izz="689649.10160904"/>
-      <!-- <inertia ixx="0" ixy="0" ixz="0" iyy="0" iyz="0" izz="0"/> -->
-    </inertial>
-    </link>
-    <gazebo reference="base_link">
-        <material>Gazebo/Yellow</material>
-    </gazebo>
+    <xacro:base_link xyz="0 0 0" rpy="0 1.57 0"></xacro:base_link>
     <!--
 // 2:right upper 1->2
@@ -67,15 +39,13 @@
 -->
     <!-- ${x}-0.32 ${y}-0.06 ${z}+0.1 -->
-    <xacro:thruster_CCW id="1" parent="base_link" xyz="0.445 -0.54 0.25" rpy="0 0 0" axis="0 0 -1">
+    <xacro:thruster_CCW id="1" parent="base_link" xyz="0.25 0.32 -0.17" rpy="0 0 0" axis="0 0 -1">
     </xacro:thruster_CCW>
-    <xacro:thruster_CW id="2" parent="base_link" xyz="0.06 -0.54 0.25" rpy="0 0 0" axis="0 0 1">
+    <xacro:thruster_CW id="2" parent="base_link" xyz="0.25 -0.32 -0.17" rpy="0 0 0" axis="0 0 1">
     </xacro:thruster_CW>
-    <xacro:thruster_CW id="4" parent="base_link" xyz="0.445 -0.32 0.25" rpy="0 0 0" axis="0 0 1">
+    <xacro:thruster_CW id="4" parent="base_link" xyz="-0.25 0.32 -0.17" rpy="0 0 0" axis="0 0 1">
     </xacro:thruster_CW>
-    <xacro:thruster_CCW id="3" parent="base_link" xyz="0.06 -0.32 0.25" rpy="0 0 0" axis="0 0 -1" >
+    <xacro:thruster_CCW id="3" parent="base_link" xyz="-0.25 -0.32 -0.17" rpy="0 0 0" axis="0 0 -1" >
     </xacro:thruster_CCW>
-    <xacro:property name="x" default="-0.26"/>
-    <xacro:property name="y" default="0.43"/>
-    <xacro:thruster_CCW id="5" parent="base_link" xyz="0.41 -0.68 0.17" rpy="0 1.57 0.785398" axis="0 0 -1">
+    <!-- <xacro:thruster_CCW id="5" parent="base_link" xyz="0.41 -0.68 0.17" rpy="0 1.57 0.785398" axis="0 0 -1">
     </xacro:thruster_CCW>
     <xacro:thruster_CW id="6" parent="base_link" xyz="0.11 -0.68 0.17" rpy="0 1.57 2.35619" axis="0 0 1">
@@ -84,8 +54,8 @@
     </xacro:thruster_CCW>
     <xacro:thruster_CW id="8" parent="base_link" xyz="0.41 -0.18 0.17" rpy="0 1.57 -0.785398" axis="0 0 1">
-    </xacro:thruster_CW>
-    <xacro:camera id="1" parent="base_link" xyz="0.255 -0.68 0.25" rpy="0 0 -1.57">
+    </xacro:thruster_CW> -->
+    <xacro:camera id="1" parent="base_link" xyz="0.3 0 0" rpy="0 0 0">
     </xacro:camera>
-    <xacro:imu id="1" parent="base_link" xyz="0.24 -0.4 0.25" rpy="0 0 -1.57">
+    <xacro:imu id="1" parent="base_link" xyz="0 0 0.15" rpy="0 0 -1.57">
     </xacro:imu>
     <gazebo>
@@ -99,9 +69,9 @@
       <descriptionParam>robot_description</descriptionParam>
       <alwaysOn>true</alwaysOn>
-      <surface>0 0 0</surface>
+      <surface>0 0 40</surface>
       <updateRate>.001</updateRate>
       <link name='base_link'>
         <buoyancy>
-          <compensation>0</compensation>
+          <compensation>0.0</compensation>
           <origin xyz="0 0 0"/>
         </buoyancy>
@@ -109,3 +79,12 @@
     </plugin>
   </gazebo>
+    <!-- <gazebo>
+     <plugin name="BuoyancyPlugin" filename="libBuoyancyPlugin.so">
+      <fluid_density>1000</fluid_density>
+      <link name="base_link">
+        <volume>0.03</volume>
+        <center_of_volume>0 0 0</center_of_volume>
+      </link>
+    </plugin>
+  </gazebo> -->
 </robot>
