Commit message: PID gyro close tuned

File: calypso-simulator/calypso_sim/model/chasis.urdf.xacro (robot description, xacro)
@@ -16,7 +16,11 @@
       <origin xyz="${xyz}" rpy="${rpy}"/>
     </collision>
+    <!-- <inertial>
+      <mass value="37"/>
+      <inertia ixx="1002084.26190628" ixy="-0.00000934" ixz="-0.00004849" iyy="1472890.49211890" iyz="1402.25179064" izz="689649.10160904"/>
+    </inertial> -->
     <inertial>
       <mass value="37"/>
-      <inertia ixx="1002084.26190628" ixy="-0.00000934" ixz="-0.00004849" iyy="1472890.49211890" iyz="1402.25179064" izz="689649.10160904"/>
+      <inertia ixx="-0.00000934" ixy="-0.00000934" ixz="-0.00000934" iyy="-0.00000934" iyz="-0.00000934" izz="-0.00000934"/>
     </inertial>
   </link>
